File: cad/hec-base/HEC-Bus-Port.sch (KiCad schematic (older format))
At the start: 34 parts

Commit message: Power-Management schematics input and dimensioning done.
Connections:
- net HEC_Data_in renamed HEC_Bitstream_in
- net HEC_Data_out renamed HEC_Bitstream_out
Changed lines of the file:
@@
 $Descr A3 16535 11693
 encoding utf-8
-Sheet 2 2
+Sheet 2 3
 Title "Marienkäfer HEC-Basis-Bord"
 Date "2020-12-28"
@@
 	3800 8250 3800 8050
 Text HLabel 1800 8150 0    50   Input ~ 0
-HEC_Data_out
+HEC_Bitstream_out
 Wire Wire Line
 	4050 7950 3450 7950
 Text HLabel 1800 7950 0    50   Output ~ 0
-HEC_Data_in
+HEC_Bitstream_in
 $Comp
 L 74xGxx:74AUP1G57 IC?

Commit message: MCU-, Crypto- und One-Wire-Teil erstellt und dimensioniert, ERC bestanden, SLP geplottet, Footprints nur teilweise zugewiesen.
Parts:
- C302, C303, C304, C305: renamed from C?; footprint (none) -> Capacitor_SMD:C_0603_1608Metric
- D301, D304: renamed from D?; footprint (none) -> LED_SMD:LED_0603_1608Metric
- D302: renamed from D?; footprint (none) -> Package_TO_SOT_SMD:SOT-23
- D303: renamed from D?; value D -> MBRS140; footprint (none) -> Diode_SMD:D_SMB
- D305: renamed from D?; footprint (none) -> Diode_SMD:D_SMB
- IC301: renamed from IC?; footprint (none) -> Package_SO:SO-8_3.9x4.9mm_P1.27mm
- IC302: renamed from IC?; footprint (none) -> Package_TO_SOT_SMD:SOT-363_SC-70-6
- J301, J303: renamed from J?; value steckbare Schraubklemme -> AKL-166-03; footprint (none) -> TerminalBlock_MetzConnect:TerminalBlock_MetzConnect_Type059_RT06303HBWC_1x03_P3.50mm_Horizontal
- J304: renamed from J?; value steckbare Schraubklemme -> AKL-166-02; footprint (none) -> TerminalBlock_MetzConnect:TerminalBlock_MetzConnect_Type059_RT06302HBWC_1x02_P3.50mm_Horizontal
- gave numbers to parts that had none: 20
Other:
- moved on the sheet: C301, C302, C303, C304, C305, D301, D302, D303, D304, D305, E301, E302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

Commit message: MT-Marienkaefer: Footprints fertig zugewiesen.
Parts:
- removed F302, F303: Fuse_Small, symbol Device:Polyfuse_Small
- added F302, F303: ESKA BSMD1206-SS0.5, Resistor_SMD:R_1206_3216Metric, symbol Device:Fuse_Small
- E301, E302, E303, E304, E305: footprint (none) -> SparkGaps_MT:SparkGap_3pin_0.67x0.5mm
- F301: value Fuse_Small -> ESKA BSMD1206-SS0.5; footprint (none) -> Resistor_SMD:R_1206_3216Metric; symbol Device:Polyfuse_Small -> Device:Fuse_Small
- L301, L302: footprint (none) -> Inductor_SMD:L_CommonMode_Wuerth_WE-SL2
- R303, R304, R306, R307, R308: footprint (none) -> Resistor_SMD:R_0603_1608Metric
Connections:
- net GND: now also F301.1, F302.1; no longer F301.2
- net at J304.1 (Pin_1): now also F303.2
- net at C302.2, D305.2 (A2), E305.1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: now also F303.1
- net at J303.1 (Pin_1): now also F302.2
- net at J301.1 (Pin_1): now also F301.2; no longer F301.1
Other:
- moved on the sheet: E305, J301, J303, J304
Changed lines of the file:
@@
 L Connector:Screw_Terminal_01x02 J304
 U 1 1 5FEA1E39
-P 11400 6600
-F 0 "J304" H 11350 6350 50  0000 L CNN
-F 1 "AKL-166-02" H 11600 6350 50  0000 L CNN
-F 2 "TerminalBlock_MetzConnect:TerminalBlock_MetzConnect_Type059_RT06302HBWC_1x02_P3.50mm_Horizontal" H 11400 6600 50  0001 C CNN
-F 3 "~" H 11400 6600 50  0001 C CNN
-	1    11400 6600
+P 11850 6600
+F 0 "J304" H 11800 6350 50  0000 L CNN
+F 1 "AKL-166-02" H 12050 6350 50  0000 L CNN
+F 2 "TerminalBlock_MetzConnect:TerminalBlock_MetzConnect_Type059_RT06302HBWC_1x02_P3.50mm_Horizontal" H 11850 6600 50  0001 C CNN
+F 3 "~" H 11850 6600 50  0001 C CNN
+	1    11850 6600
 	1    0    0    1
 $EndComp
-Text Notes 11550 5750 0    50   ~ 0
+Text Notes 12000 5750 0    50   ~ 0
 Bus-Ground
 $Comp
@@
 F 0 "L302" H 7150 6600 50  0000 C CNN
 F 1 "WE 744220" H 7400 6400 50  0000 C CNN
-F 2 "" H 7450 6600 50  0001 C CNN
+F 2 "Inductor_SMD:L_CommonMode_Wuerth_WE-SL2" H 7450 6600 50  0001 C CNN
 F 3 "~" H 7450 6600 50  0001 C CNN
 	1    7450 6600
@@
 F 0 "L301" H 7150 6200 50  0000 C CNN
 F 1 "WE 744227" H 7400 6450 50  0000 C CNN
-F 2 "" H 7450 6200 50  0001 C CNN
+F 2 "Inductor_SMD:L_CommonMode_Wuerth_WE-SL2" H 7450 6200 50  0001 C CNN
 F 3 "~" H 7450 6200 50  0001 C CNN
 	1    7450 6200
@@
 	8000 5900 9600 5900
 Wire Wire Line
-	11200 5800 10000 5800
+	11650 5800 10000 5800
 Wire Wire Line
 	7900 5800 7900 6100
@@
 	1    0    0    -1
 $EndComp
-$Comp
-L Device:Polyfuse_Small F303
-U 1 1 5FEB6B11
-P 10800 6600
-F 0 "F303" V 11000 6600 50  0000 C CNN
-F 1 "Fuse_Small" V 10900 6600 50  0000 C CNN
-F 2 "" H 10800 6600 50  0001 C CNN
-F 3 "~" H 10800 6600 50  0001 C CNN
-	1    10800 6600
-	0    1    1    0
-$EndComp
 Connection ~ 7050 6950
-$Comp
-L Device:Polyfuse_Small F302
-U 1 1 5FEBAF89
-P 10900 5700
-F 0 "F302" V 10700 5700 50  0000 C CNN
-F 1 "Fuse_Small" V 10800 5700 50  0000 C CNN
-F 2 "" H 10900 5700 50  0001 C CNN
-F 3 "~" H 10900 5700 50  0001 C CNN
-	1    10900 5700
-	0    1    1    0
-$EndComp
 Wire Wire Line
 	6750 5650 6750 5600
@@
 	9350 6950 9350 5700
 Connection ~ 9350 5700
-Text Notes 11550 6550 0    50   ~ 0
+Text Notes 12000 6550 0    50   ~ 0
 Versorgung + (24V)
-Text Notes 11550 6650 0    50   ~ 0
+Text Notes 12000 6650 0    50   ~ 0
 Versorgung - (0V)
-Text Notes 11550 5950 0    50   ~ 0
+Text Notes 12000 5950 0    50   ~ 0
 HEC-Bus B
-Text Notes 11550 5850 0    50   ~ 0
+Text Notes 12000 5850 0    50   ~ 0
 HEC-Bus A
 $Comp
 L Connector:Screw_Terminal_01x03 J303
 U 1 1 5FEE6F28
-P 11400 5800
-F 0 "J303" H 11350 6050 50  0000 L CNN
-F 1 "AKL-166-03" H 11600 6050 50  0000 L CNN
-F 2 "TerminalBlock_MetzConnect:TerminalBlock_MetzConnect_Type059_RT06303HBWC_1x03_P3.50mm_Horizontal" H 11400 5800 50  0001 C CNN
-F 3 "~" H 11400 5800 50  0001 C CNN
-	1    11400 5800
-	1    0    0    -1
-$EndComp
-Text Notes 11550 5100 0    50   ~ 0
+P 11850 5800
+F 0 "J303" H 11800 6050 50  0000 L CNN
+F 1 "AKL-166-03" H 12050 6050 50  0000 L CNN
+F 2 "TerminalBlock_MetzConnect:TerminalBlock_MetzConnect_Type059_RT06303HBWC_1x03_P3.50mm_Horizontal" H 11850 5800 50  0001 C CNN
+F 3 "~" H 11850 5800 50  0001 C CNN
+	1    11850 5800
+	1    0    0    -1
+$EndComp
+Text Notes 12000 5100 0    50   ~ 0
 Bus-Ground
 $Comp
-L Device:Polyfuse_Small F301
+L Device:Fuse_Small F301
 U 1 1 5FEEED7B
-P 10900 5050
-F 0 "F301" V 10700 5050 50  0000 C CNN
-F 1 "Fuse_Small" V 10800 5050 50  0000 C CNN
-F 2 "" H 10900 5050 50  0001 C CNN
-F 3 "~" H 10900 5050 50  0001 C CNN
-	1    10900 5050
-	0    1    1    0
-$EndComp
-Text Notes 11550 5300 0    50   ~ 0
+P 11100 5050
+F 0 "F301" H 11100 5250 50  0000 C CNN
+F 1 "ESKA BSMD1206-SS0.5" H 11100 5150 50  0000 C CNN
+F 2 "Resistor_SMD:R_1206_3216Metric" H 11100 5050 50  0001 C CNN
+F 3 "~" H 11100 5050 50  0001 C CNN
+	1    11100 5050
+	1    0    0    -1
+$EndComp
+Text Notes 12000 5300 0    50   ~ 0
 HEC-Bus B
-Text Notes 11550 5200 0    50   ~ 0
+Text Notes 12000 5200 0    50   ~ 0
 HEC-Bus A
 $Comp
 L Connector:Screw_Terminal_01x03 J301
 U 1 1 5FEEED89
-P 11400 5150
-F 0 "J301" H 11350 5400 50  0000 L CNN
-F 1 "AKL-166-03" H 11600 5400 50  0000 L CNN
-F 2 "TerminalBlock_MetzConnect:TerminalBlock_MetzConnect_Type059_RT06303HBWC_1x03_P3.50mm_Horizontal" H 11400 5150 50  0001 C CNN
-F 3 "~" H 11400 5150 50  0001 C CNN
-	1    11400 5150
+P 11850 5150
+F 0 "J301" H 11800 5400 50  0000 L CNN
+F 1 "AKL-166-03" H 12050 5400 50  0000 L CNN
+F 2 "TerminalBlock_MetzConnect:TerminalBlock_MetzConnect_Type059_RT06303HBWC_1x03_P3.50mm_Horizontal" H 11850 5150 50  0001 C CNN
+F 3 "~" H 11850 5150 50  0001 C CNN
+	1    11850 5150
 	1    0    0    -1
 $EndComp
@@
 F 0 "R307" H 5770 6496 50  0000 L CNN
 F 1 "2k4" H 5770 6405 50  0000 L CNN
-F 2 "" V 5630 6450 50  0001 C CNN
+F 2 "Resistor_SMD:R_0603_1608Metric" V 5630 6450 50  0001 C CNN
 F 3 "~" H 5700 6450 50  0001 C CNN
 	1    5700 6450
@@
 F 0 "R304" H 5120 5446 50  0000 L CNN
 F 1 "2k4" H 5120 5355 50  0000 L CNN
-F 2 "" V 4980 5400 50  0001 C CNN
+F 2 "Resistor_SMD:R_0603_1608Metric" V 4980 5400 50  0001 C CNN
 F 3 "~" H 5050 5400 50  0001 C CNN
 	1    5050 5400
@@
 F 0 "R306" V 5700 6000 50  0000 C CNN
 F 1 "4k7" V 5600 6000 50  0000 C CNN
-F 2 "" V 5330 6000 50  0001 C CNN
+F 2 "Resistor_SMD:R_0603_1608Metric" V 5330 6000 50  0001 C CNN
 F 3 "~" H 5400 6000 50  0001 C CNN
 	1    5400 6000
@@
 F 0 "R303" V 2650 5050 50  0000 L CNN
 F 1 "330R" V 2750 5050 50  0000 L CNN
-F 2 "" V 2780 5150 50  0001 C CNN
+F 2 "Resistor_SMD:R_0603_1608Metric" V 2780 5150 50  0001 C CNN
 F 3 "~" H 2850 5150 50  0001 C CNN
 	1    2850 5150
@@
 F 0 "R308" H 3300 7000 50  0000 L CNN
 F 1 "330R" H 3300 6900 50  0000 L CNN
-F 2 "" V 3130 6950 50  0001 C CNN
+F 2 "Resistor_SMD:R_0603_1608Metric" V 3130 6950 50  0001 C CNN
 F 3 "~" H 3200 6950 50  0001 C CNN
 	1    3200 6950
@@
 	8750 6700 8750 6600
 Wire Wire Line
-	10700 6600 10500 6600
+	10900 6600 10700 6600
 Wire Wire Line
 	9500 6600 9500 6700
@@
 L Device:SPARK_GAP E305
 U 1 1 5FFD4BDB
-P 10800 6450
-F 0 "E305" H 10800 6548 50  0000 C CNN
-F 1 "SPARK_GAP" H 10800 6549 50  0001 C CNN
-F 2 "" H 10800 6380 50  0001 C CNN
-F 3 "~" V 10800 6450 50  0001 C CNN
-	1    10800 6450
-	1    0    0    -1
-$EndComp
-Wire Wire Line
-	11000 6450 11050 6450
-Wire Wire Line
-	11050 6450 11050 6500
-Wire Wire Line
-	11050 6500 11200 6500
+P 11000 6450
+F 0 "E305" H 11000 6548 50  0000 C CNN
+F 1 "SPARK_GAP" H 11000 6549 50  0001 C CNN
+F 2 "SparkGaps_MT:SparkGap_3pin_0.67x0.5mm" H 11000 6380 50  0001 C CNN
+F 3 "~" V 11000 6450 50  0001 C CNN
+	1    11000 6450
+	1    0    0    -1
+$EndComp
+Wire Wire Line
+	11200 6450 11250 6450
+Wire Wire Line
+	11250 6450 11250 6500
+Wire Wire Line
+	11250 6500 11650 6500
 $Comp
 L Device:SPARK_GAP E303
@@
 F 0 "E303" H 10250 5698 50  0000 C CNN
 F 1 "SPARK_GAP" H 10250 5699 50  0001 C CNN
-F 2 "" H 10250 5530 50  0001 C CNN
+F 2 "SparkGaps_MT:SparkGap_3pin_0.67x0.5mm" H 10250 5530 50  0001 C CNN
 F 3 "~" V 10250 5600 50  0001 C CNN
 	1    10250 5600
@@
 F 0 "E304" H 10250 5850 50  0000 C CNN
 F 1 "SPARK_GAP" H 10250 5850 50  0001 C CNN
-F 2 "" H 10250 5880 50  0001 C CNN
+F 2 "SparkGaps_MT:SparkGap_3pin_0.67x0.5mm" H 10250 5880 50  0001 C CNN
 F 3 "~" V 10250 5950 50  0001 C CNN
 	1    10250 5950
@@
 Connection ~ 10000 5900
 Wire Wire Line
-	10000 5900 11200 5900
+	10000 5900 11650 5900
 $Comp
 L Device:SPARK_GAP E301
@@
 F 0 "E301" H 10250 5098 50  0000 C CNN
 F 1 "SPARK_GAP" H 10250 5099 50  0001 C CNN
-F 2 "" H 10250 4930 50  0001 C CNN
+F 2 "SparkGaps_MT:SparkGap_3pin_0.67x0.5mm" H 10250 4930 50  0001 C CNN
 F 3 "~" V 10250 5000 50  0001 C CNN
 	1    10250 5000
@@
 F 0 "E302" H 10250 5200 50  0000 C CNN
 F 1 "SPARK_GAP" H 10250 5200 50  0001 C CNN
-F 2 "" H 10250 5230 50  0001 C CNN
+F 2 "SparkGaps_MT:SparkGap_3pin_0.67x0.5mm" H 10250 5230 50  0001 C CNN
 F 3 "~" V 10250 5300 50  0001 C CNN
 	1    10250 5300
@@
 Connection ~ 10000 5250
 Wire Wire Line
-	10000 5250 11200 5250
+	10000 5250 11650 5250
 Wire Wire Line
 	10050 5000 10000 5000
@@
 	10000 5000 10000 5150
 Connection ~ 10000 5150
-Wire Wire Line
-	10000 5150 11200 5150
 $Comp
 L power:GNDD #PWR0310
@@
 $EndComp
 Wire Wire Line
-	10900 6600 11200 6600
-Wire Wire Line
-	10500 6450 10500 6600
-Wire Wire Line
-	10500 6450 10600 6450
-Connection ~ 10500 6600
-Wire Wire Line
-	10500 6600 9500 6600
-Wire Wire Line
-	11000 5700 11200 5700
+	11100 6600 11650 6600
+Wire Wire Line
+	10700 6450 10700 6600
+Wire Wire Line
+	10700 6450 10800 6450
+Connection ~ 10700 6600
+Wire Wire Line
+	10700 6600 9500 6600
+Wire Wire Line
+	11200 5700 11650 5700
 Wire Wire Line
 	10500 5600 10500 5700
 Connection ~ 10500 5700
 Wire Wire Line
-	10500 5700 10800 5700
+	10500 5700 11000 5700
 Wire Wire Line
 	10500 5700 10500 5950
@@
 	9350 5050 10500 5050
 Wire Wire Line
-	10800 5050 10500 5050
-Wire Wire Line
-	11200 5050 11000 5050
+	11000 5050 10500 5050
+Wire Wire Line
+	11650 5050 11200 5050
 Text Notes 9850 7050 0    50   ~ 0
 Funkenstrecken so dicht wie möglich an die Klemmen!
@@
 Wire Wire Line
 	8150 6500 9250 6500
-Connection ~ 11050 6500
+Connection ~ 11250 6500
 Wire Wire Line
 	9500 6250 9500 6500
@@
 Connection ~ 9500 6500
 Wire Wire Line
-	9500 6500 11050 6500
+	9500 6500 11250 6500
 Wire Wire Line
 	7650 6500 7850 6500
@@
 Wire Wire Line
 	1750 7050 1750 7200
+Wire Wire Line
+	10000 5150 11650 5150
+$Comp
+L Device:Fuse_Small F302
+U 1 1 5FF99D46
+P 11100 5700
+F 0 "F302" H 11100 5900 50  0000 C CNN
+F 1 "ESKA BSMD1206-SS0.5" H 11100 5800 50  0000 C CNN
+F 2 "Resistor_SMD:R_1206_3216Metric" H 11100 5700 50  0001 C CNN
+F 3 "~" H 11100 5700 50  0001 C CNN
+	1    11100 5700
+	1    0    0    -1
+$EndComp
+$Comp
+L Device:Fuse_Small F303
+U 1 1 5FF9A244
+P 11000 6600
+F 0 "F303" H 11000 6500 50  0000 C CNN
+F 1 "ESKA BSMD1206-SS0.5" H 11000 6400 50  0000 C CNN
+F 2 "Resistor_SMD:R_1206_3216Metric" H 11000 6600 50  0001 C CNN
+F 3 "~" H 11000 6600 50  0001 C CNN
+	1    11000 6600
+	1    0    0    -1
+$EndComp
 $EndSCHEMATC

Commit message: Entflochtene Leiterplatte mit Schaltplan speichern.
Parts:
- removed F303: ESKA BSMD1206-SS0.5, Resistor_SMD:R_1206_3216Metric, symbol Device:Fuse_Small
- added unit 2 of IC302
- D302: symbol Device:D_TVS_x2_AAC -> Device:D_TVS_Dual_AAC
- E301, E302, E303, E304, E305: symbol Device:SPARK_GAP -> Device:SparkGap
- IC302: symbol 74xGxx:74AUP1G57 -> Logic_74xGxx_MT:74LVC1G57
- L301, L302: symbol Device:L_Core_Ferrite_Coupled -> Device:L_Ferrite_Coupled_1423
Connections:
- net +5V: no longer C303.1, C304.1, IC301.8 (VCC), IC302.5 (VCC), R303.2, R304.1
- net at J304.1 (Pin_1): now also E305.1, F302.2
- net at D302.1 (A1), IC301.7 (B), R306.1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: now also L301.2; no longer L301.3
- net at D303.1 (K): now also L302.4; no longer L302.2
- net at C302.2, D305.2 (A2): now also F302.1, L302.3; no longer E305.1, L302.4
- net at E301.1, E303.1, J301.2 (Pin_2)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: now also L301.4; no longer L301.2
- net at E302.1, E304.1, J301.3 (Pin_3)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: now also L301.3; no longer L301.4
- net at J303.1 (Pin_1): now also E301.2, E302.2, E303.2, E304.2, F301.2, J301.1 (Pin_1); no longer F302.2
- net GND renamed GNDD
- net GNDD: now also L302.2, IC302.2 (GND); no longer E301.2, E302.2, E303.2, E304.2, F302.1, IC302.2 (GND), L302.3
- net HEC_Bitstream_in renamed HEC_Bitstream_in_FV
- net HEC_Bitstream_out renamed HEC_Bitstream_out_FT
- new net 5V: C303.1, C304.1, IC301.8 (VCC), IC302.5 (VCC), R303.2, R304.1
Other:
- note added: "Inverter\n(2-Input NOR)"
- note added: "TODO:\no Symbol für stromkompensierte Drosseln überprüfen\n"
- note removed: "TODO:\no Symbol für stromkompensierte Drosseln überprüfen\no LED-Typen festlegen\no Polyfuse festlegen\no"
- moved on the sheet: C303, C305, D302, E301, E302, E303, E304, F301, F302
