File: cad/hec-base/mcu.sch (KiCad schematic (older format))
At the start: 29 parts, among them IC205 STM32F103C8Tx, J401 Micromatch 6p, J402 Cortex-Debug WSL 2x5 RM1.27

Commit message: MT-Marienkaefer: Footprints fertig zugewiesen.
Parts:
- J402: footprint (none) -> Connector_PinHeader_1.27mm:PinHeader_2x05_P1.27mm_Vertical_SMD
- R401, R402, R403, R404, R405, R406, R407, R408, R409, R410, R411: footprint (none) -> Resistor_SMD:R_0603_1608Metric
- TP401, TP402, TP403, TP404, TP405, TP406: footprint (none) -> TestPoint:TestPoint_Pad_D1.0mm
- XTAL401: footprint (none) -> Crystal:Crystal_SMD_HC49-SD
Changed lines of the file:
@@
 F 0 "XTAL401" H 5450 10118 50  0000 C CNN
 F 1 "HC49-SMD 8,000 MHz" H 5450 10027 50  0000 C CNN
-F 2 "" H 5450 9850 50  0001 C CNN
+F 2 "Crystal:Crystal_SMD_HC49-SD" H 5450 9850 50  0001 C CNN
 F 3 "~" H 5450 9850 50  0001 C CNN
 	1    5450 9850
@@
 F 0 "R411" H 3070 9896 50  0000 L CNN
 F 1 "4k7" H 3070 9805 50  0000 L CNN
-F 2 "" V 2930 9850 50  0001 C CNN
+F 2 "Resistor_SMD:R_0603_1608Metric" V 2930 9850 50  0001 C CNN
 F 3 "~" H 3000 9850 50  0001 C CNN
 	1    3000 9850
@@
 F 0 "TP401" H 11308 7668 50  0000 L CNN
 F 1 "TMS" H 11308 7577 50  0000 L CNN
-F 2 "" H 11450 7550 50  0001 C CNN
+F 2 "TestPoint:TestPoint_Pad_D1.0mm" H 11450 7550 50  0001 C CNN
 F 3 "~" H 11450 7550 50  0001 C CNN
 	1    11250 7550
@@
 F 0 "TP404" H 12208 7668 50  0000 L CNN
 F 1 "TCK" H 12208 7577 50  0000 L CNN
-F 2 "" H 12350 7550 50  0001 C CNN
+F 2 "TestPoint:TestPoint_Pad_D1.0mm" H 12350 7550 50  0001 C CNN
 F 3 "~" H 12350 7550 50  0001 C CNN
 	1    12150 7550
@@
 F 0 "TP402" H 11608 7668 50  0000 L CNN
 F 1 "TRST" H 11608 7577 50  0000 L CNN
-F 2 "" H 11750 7550 50  0001 C CNN
+F 2 "TestPoint:TestPoint_Pad_D1.0mm" H 11750 7550 50  0001 C CNN
 F 3 "~" H 11750 7550 50  0001 C CNN
 	1    11550 7550
@@
 F 0 "TP403" H 11908 7668 50  0000 L CNN
 F 1 "SRST" H 11908 7577 50  0000 L CNN
-F 2 "" H 12050 7550 50  0001 C CNN
+F 2 "TestPoint:TestPoint_Pad_D1.0mm" H 12050 7550 50  0001 C CNN
 F 3 "~" H 12050 7550 50  0001 C CNN
 	1    11850 7550
@@
 F 0 "TP405" H 12508 7668 50  0000 L CNN
 F 1 "TDI" H 12508 7577 50  0000 L CNN
-F 2 "" H 12650 7550 50  0001 C CNN
+F 2 "TestPoint:TestPoint_Pad_D1.0mm" H 12650 7550 50  0001 C CNN
 F 3 "~" H 12650 7550 50  0001 C CNN
 	1    12450 7550
@@
 F 0 "TP406" H 12808 7668 50  0000 L CNN
 F 1 "TDO" H 12808 7577 50  0000 L CNN
-F 2 "" H 12950 7550 50  0001 C CNN
+F 2 "TestPoint:TestPoint_Pad_D1.0mm" H 12950 7550 50  0001 C CNN
 F 3 "~" H 12950 7550 50  0001 C CNN
 	1    12750 7550
@@
 F 0 "J402" H 10550 8367 50  0000 C CNN
 F 1 "Cortex-Debug WSL 2x5 RM1.27" H 10550 8276 50  0000 C CNN
-F 2 "" H 10500 7950 50  0001 C CNN
+F 2 "Connector_PinHeader_1.27mm:PinHeader_2x05_P1.27mm_Vertical_SMD" H 10500 7950 50  0001 C CNN
 F 3 "~" H 10500 7950 50  0001 C CNN
 	1    10500 7950
@@
 F 0 "R409" H 3170 6596 50  0000 L CNN
 F 1 "120R" H 3170 6505 50  0000 L CNN
-F 2 "" V 3030 6550 50  0001 C CNN
+F 2 "Resistor_SMD:R_0603_1608Metric" V 3030 6550 50  0001 C CNN
 F 3 "~" H 3100 6550 50  0001 C CNN
 	1    3100 6550
@@
 F 0 "R410" H 3620 6596 50  0000 L CNN
 F 1 "120R" H 3620 6505 50  0000 L CNN
-F 2 "" V 3480 6550 50  0001 C CNN
+F 2 "Resistor_SMD:R_0603_1608Metric" V 3480 6550 50  0001 C CNN
 F 3 "~" H 3550 6550 50  0001 C CNN
 	1    3550 6550
@@
 F 0 "R408" H 7170 4696 50  0000 L CNN
 F 1 "4k7" H 7170 4605 50  0000 L CNN
-F 2 "" V 7030 4650 50  0001 C CNN
+F 2 "Resistor_SMD:R_0603_1608Metric" V 7030 4650 50  0001 C CNN
 F 3 "~" H 7100 4650 50  0001 C CNN
 	1    7100 4650
@@
 F 0 "R401" H 5950 2350 50  0000 L CNN
 F 1 "4k7" H 6020 2155 50  0000 L CNN
-F 2 "" V 5880 2200 50  0001 C CNN
+F 2 "Resistor_SMD:R_0603_1608Metric" V 5880 2200 50  0001 C CNN
 F 3 "~" H 5950 2200 50  0001 C CNN
 	1    5950 2200
@@
 F 0 "R402" H 6250 2350 50  0000 L CNN
 F 1 "4k7" H 6320 2155 50  0000 L CNN
-F 2 "" V 6180 2200 50  0001 C CNN
+F 2 "Resistor_SMD:R_0603_1608Metric" V 6180 2200 50  0001 C CNN
 F 3 "~" H 6250 2200 50  0001 C CNN
 	1    6250 2200
@@
 F 0 "R404" H 6850 2350 50  0000 L CNN
 F 1 "4k7" H 6920 2155 50  0000 L CNN
-F 2 "" V 6780 2200 50  0001 C CNN
+F 2 "Resistor_SMD:R_0603_1608Metric" V 6780 2200 50  0001 C CNN
 F 3 "~" H 6850 2200 50  0001 C CNN
 	1    6850 2200
@@
 F 0 "R403" H 6550 2350 50  0000 L CNN
 F 1 "4k7" H 6620 2155 50  0000 L CNN
-F 2 "" V 6480 2200 50  0001 C CNN
+F 2 "Resistor_SMD:R_0603_1608Metric" V 6480 2200 50  0001 C CNN
 F 3 "~" H 6550 2200 50  0001 C CNN
 	1    6550 2200
@@
 F 0 "R406" H 5200 3850 50  0000 L CNN
 F 1 "1k" H 5270 3655 50  0000 L CNN
-F 2 "" V 5130 3700 50  0001 C CNN
+F 2 "Resistor_SMD:R_0603_1608Metric" V 5130 3700 50  0001 C CNN
 F 3 "~" H 5200 3700 50  0001 C CNN
 	1    5200 3700
@@
 F 0 "R407" H 5500 3850 50  0000 L CNN
 F 1 "1k" H 5570 3655 50  0000 L CNN
-F 2 "" V 5430 3700 50  0001 C CNN
+F 2 "Resistor_SMD:R_0603_1608Metric" V 5430 3700 50  0001 C CNN
 F 3 "~" H 5500 3700 50  0001 C CNN
 	1    5500 3700
@@
 F 0 "R405" H 4900 3850 50  0000 L CNN
 F 1 "4k7" H 4970 3655 50  0000 L CNN
-F 2 "" V 4830 3700 50  0001 C CNN
+F 2 "Resistor_SMD:R_0603_1608Metric" V 4830 3700 50  0001 C CNN
 F 3 "~" H 4900 3700 50  0001 C CNN
 	1    4900 3700

Commit message: Entflochtene Leiterplatte mit Schaltplan speichern.
Parts:
- added JP404, JP405: SolderJumper_3_Open, Jumper:SolderJumper-3_P1.3mm_Open_RoundedPad1.0x1.5mm_NumberLabels, symbol Jumper:SolderJumper_3_Open
- J401: value Micromatch 6p -> Tag-Connect 2x3; footprint Connectors_MicroMatch_MT:ConnectorMicromatch-6-SMD-polarized -> Tag-Connect:Tag-Connect_TC2030-IDC-NL_2x03_P1.27mm_Vertical; symbol Connector_Generic:Conn_02x03_Odd_Even -> Tag-Connect:TC2030-IDC-console
- J402: value Cortex-Debug WSL 2x5 RM1.27 -> Tag-Connect 2x5; footprint Connector_PinHeader_1.27mm:PinHeader_2x05_P1.27mm_Vertical_SMD -> Tag-Connect:Tag-Connect_TC2050-IDC-NL_2x05_P1.27mm_Vertical
Connections:
- net +3V3: now also JP404.3 (B); no longer R408.1
- net +5V: now also R408.1
- net GNDD: now also JP404.1 (A), JP405.3 (B); no longer J402.5 (Pin_5), J402.9 (Pin_9)
- net VccSNS3V3: now also IC205.15 (PA5); no longer IC205.16 (PA6)
- net VccSNS5V: now also IC205.16 (PA6); no longer IC205.15 (PA5)
- net ~TRST~: now also JP405.1 (A)
- net HEC-Bitstream-in renamed HEC-Bitstream-in-FT
- net HEC-Bitstream-out renamed HEC-Bitstream-out-FT
- new net: J402.5 (Pin_5), JP404.2 (C)
- new net: J402.9 (Pin_9), JP405.2 (C)
Other:
- note added: "Pin 5 should be grounded, but some debuggers \nsupply 5V here or 3V3 (i.e. STLINK/V2).\nPin 7 is a Key-Pin for SWDIO, normally \nremove (pull out), RTCK for JTAG is not available,\nPin 9 can be grounded for SWDIO, but \nconnected to ~TRST~ for JTAG."
- note added: "TODO:\no STM32F0xx als Alternativ-Bestückung prüfen/vorsehen, entsprechend Pins beschalten\no STM32F30x als Alternativ-Bestückung prüfen/vorsehen, entsprechend Pins beschalten\no STM32F7xx als Alternativ-Bestückung prüfen/vorsehen, entsprechend Pins beschalten"
- note removed: "Pin 7 ist ein Key-Pin, \nnormal entfernen (ziehen)"
- note removed: "oder \nWSL 2x3 RM2.54"
- moved on the sheet: C401, J402, JP403, R408
