File: cad/hec-base/one-wire.sch (KiCad schematic (older format))
At the start: 19 parts, among them IC501 DS2482S-100, IC502 DS18B20, IC503 DS28E25, Q501 BSS123, T501 BSS84

Commit message: MT-Marienkaefer: Footprints fertig zugewiesen.
Parts:
- FL501, FL502: footprint (none) -> Filter_MT:Murata_NFE61P
- R501, R502, R503, R504, R505, R506: footprint (none) -> Resistor_SMD:R_0603_1608Metric
Changed lines of the file:
@@
 F 0 "R501" H 6020 3096 50  0000 L CNN
 F 1 "22R" H 6020 3005 50  0000 L CNN
-F 2 "" V 5880 3050 50  0001 C CNN
+F 2 "Resistor_SMD:R_0603_1608Metric" V 5880 3050 50  0001 C CNN
 F 3 "~" H 5950 3050 50  0001 C CNN
 	1    5950 3050
@@
 F 0 "R503" V 5493 4000 50  0000 C CNN
 F 1 "22R" V 5584 4000 50  0000 C CNN
-F 2 "" V 5630 4000 50  0001 C CNN
+F 2 "Resistor_SMD:R_0603_1608Metric" V 5630 4000 50  0001 C CNN
 F 3 "~" H 5700 4000 50  0001 C CNN
 	1    5700 4000
@@
 F 0 "FL502" H 6500 4417 50  0000 C CNN
 F 1 "NFE61P681B1H9L" H 6500 4326 50  0000 C CNN
-F 2 "" V 6500 4100 50  0001 C CNN
+F 2 "Filter_MT:Murata_NFE61P" V 6500 4100 50  0001 C CNN
 F 3 "http://www.murata.com/~/media/webrenewal/support/library/catalog/products/emc/emifil/c31e.ashx?la=en-gb" V 6500 4100 50  0001 C CNN
 	1    6500 4100
@@
 F 0 "FL501" H 7050 3667 50  0000 C CNN
 F 1 "NFE61P681B1H9L" H 7050 3576 50  0000 C CNN
-F 2 "" V 7050 3350 50  0001 C CNN
+F 2 "Filter_MT:Murata_NFE61P" V 7050 3350 50  0001 C CNN
 F 3 "http://www.murata.com/~/media/webrenewal/support/library/catalog/products/emc/emifil/c31e.ashx?la=en-gb" V 7050 3350 50  0001 C CNN
 	1    7050 3350
@@
 F 0 "R502" H 7870 3596 50  0000 L CNN
 F 1 "22R" H 7870 3505 50  0000 L CNN
-F 2 "" V 7730 3550 50  0001 C CNN
+F 2 "Resistor_SMD:R_0603_1608Metric" V 7730 3550 50  0001 C CNN
 F 3 "~" H 7800 3550 50  0001 C CNN
 	1    7800 3550
@@
 F 0 "R504" H 3600 4400 50  0000 L CNN
 F 1 "22R" H 3670 4205 50  0000 L CNN
-F 2 "" V 3530 4250 50  0001 C CNN
+F 2 "Resistor_SMD:R_0603_1608Metric" V 3530 4250 50  0001 C CNN
 F 3 "~" H 3600 4250 50  0001 C CNN
 	1    3600 4250
@@
 F 0 "R505" H 3900 4400 50  0000 L CNN
 F 1 "22R" H 3970 4205 50  0000 L CNN
-F 2 "" V 3830 4250 50  0001 C CNN
+F 2 "Resistor_SMD:R_0603_1608Metric" V 3830 4250 50  0001 C CNN
 F 3 "~" H 3900 4250 50  0001 C CNN
 	1    3900 4250
@@
 F 0 "R506" H 2420 5596 50  0000 L CNN
 F 1 "1k" H 2420 5505 50  0000 L CNN
-F 2 "" V 2280 5550 50  0001 C CNN
+F 2 "Resistor_SMD:R_0603_1608Metric" V 2280 5550 50  0001 C CNN
 F 3 "~" H 2350 5550 50  0001 C CNN
 	1    2350 5550

Commit message: Entflochtene Leiterplatte mit Schaltplan speichern.
Parts:
- FL501, FL502: symbol Device:EMI_Filter_LCL -> Device:Filter_EMI_LCL
- renumbered Q501 to T502
Connections:
- net +3V3 renamed 3V3
- net +5V renamed 5V
Changed lines of the file:
@@
 $Descr A4 11693 8268
 encoding utf-8
-Sheet 5 5
-Title "Marienkäfer HEC-Basis-Bord: One-Wire-Interface"
+Sheet 3 5
+Title "Marienkaefer HEC-Basis-Bord: One-Wire-Interface"
 Date ""
 Rev "0001"
@@
 	5500 4950 5500 4900
 $Comp
-L Device:EMI_Filter_LCL FL?
+L Device:Filter_EMI_LCL FL?
 U 1 1 60830233
 P 6500 4100
 AR Path="/6037F603/60830233" Ref="FL?"  Part="1"
 AR Path="/6082A275/60830233" Ref="FL502"  Part="1"
+AR Path="/60830233" Ref="FL502"  Part="1"
 F 0 "FL502" H 6500 4417 50  0000 C CNN
 F 1 "NFE61P681B1H9L" H 6500 4326 50  0000 C CNN
@@
 $EndComp
 $Comp
-L Device:EMI_Filter_LCL FL?
+L Device:Filter_EMI_LCL FL?
 U 1 1 60830241
 P 7050 3350
 AR Path="/6037F603/60830241" Ref="FL?"  Part="1"
 AR Path="/6082A275/60830241" Ref="FL501"  Part="1"
+AR Path="/60830241" Ref="FL501"  Part="1"
 F 0 "FL501" H 7050 3667 50  0000 C CNN
 F 1 "NFE61P681B1H9L" H 7050 3576 50  0000 C CNN
@@
 	1    0    0    -1
 $EndComp
-$Comp
-L power:+5V #PWR?
-U 1 1 60830247
-P 5950 2750
-AR Path="/6037F603/60830247" Ref="#PWR?"  Part="1"
-AR Path="/6082A275/60830247" Ref="#PWR0501"  Part="1"
-F 0 "#PWR0501" H 5950 2600 50  0001 C CNN
-F 1 "+5V" H 5965 2923 50  0000 C CNN
-F 2 "" H 5950 2750 50  0001 C CNN
-F 3 "" H 5950 2750 50  0001 C CNN
-	1    5950 2750
-	1    0    0    -1
-$EndComp
-Wire Wire Line
-	5950 2750 5950 2800
 Wire Wire Line
 	5950 2800 6500 2800
@@
 	1    0    0    -1
 $EndComp
-$Comp
-L power:+5V #PWR?
-U 1 1 608302CB
-P 4750 5350
-AR Path="/6037F603/608302CB" Ref="#PWR?"  Part="1"
-AR Path="/6082A275/608302CB" Ref="#PWR0505"  Part="1"
-F 0 "#PWR0505" H 4750 5200 50  0001 C CNN
-F 1 "+5V" H 4765 5523 50  0000 C CNN
-F 2 "" H 4750 5350 50  0001 C CNN
-F 3 "" H 4750 5350 50  0001 C CNN
-	1    4750 5350
-	1    0    0    -1
-$EndComp
 Wire Wire Line
 	4350 5500 4350 5450
@@
 P 2750 5700
 AR Path="/6037F603/608302E1" Ref="Q?"  Part="1"
-AR Path="/6082A275/608302E1" Ref="Q501"  Part="1"
-F 0 "Q501" V 2999 5700 50  0000 C CNN
+AR Path="/6082A275/608302E1" Ref="T502"  Part="1"
+F 0 "T502" V 2999 5700 50  0000 C CNN
 F 1 "BSS123" V 3090 5700 50  0000 C CNN
 F 2 "Package_TO_SOT_SMD:SOT-23" H 2950 5625 50  0001 L CIN
@@
 	2950 5800 3400 5800
 Connection ~ 3400 5800
-$Comp
-L power:+3V3 #PWR?
-U 1 1 608302E9
-P 2750 5050
-AR Path="/6037F603/608302E9" Ref="#PWR?"  Part="1"
-AR Path="/6082A275/608302E9" Ref="#PWR0504"  Part="1"
-F 0 "#PWR0504" H 2750 4900 50  0001 C CNN
-F 1 "+3V3" H 2765 5223 50  0000 C CNN
-F 2 "" H 2750 5050 50  0001 C CNN
-F 3 "" H 2750 5050 50  0001 C CNN
-	1    2750 5050
-	1    0    0    -1
-$EndComp
-Wire Wire Line
-	2750 5050 2750 5200
 Wire Wire Line
 	2550 5800 2350 5800
@@
 Wire Wire Line
 	2350 5200 2350 5400
-Connection ~ 2750 5200
 Wire Wire Line
 	2750 5200 2750 5500
@@
 Connection ~ 4300 2800
 Text HLabel 1700 5200 0    50   Input ~ 0
-3V
+3V3
 Wire Wire Line
 	1700 5200 2350 5200
 Connection ~ 2350 5200
+Text Label 3150 2800 0    50   ~ 0
+Vcc5V
+Text Label 1850 5200 0    50   ~ 0
+Vcc3V3
+Text Label 4750 5350 0    50   ~ 0
+Vcc5V
 $EndSCHEMATC
